Commit message: Update Robot Model for Front Plate.

File: description/robot_core.xacro (robot description, xacro)
@@ -4,42 +4,45 @@
      For more information, please see http://wiki.ros.org/sw_urdf_exporter -->
 <robot xmlns:xacro="http://www.ros.org/wiki/xacro">
-  <!-- BASE LINK -->
-  <link name="base_link">
-   <inertial>
-          <origin
-            xyz="0.067406 0.0019312 0.021326"
-            rpy="0 0 0" />
-          <mass
-            value="0.59569" />
-          <inertia
-            ixx="0.0017912"
-            ixy="7.7075E-05"
-            ixz="0.00031985"
-            iyy="0.0029313"
-            iyz="2.4441E-05"
-            izz="0.0041728" />
-   </inertial>
-   <visual>
-          <origin
-            xyz="0 0 0"
-            rpy="0 0 0" />
-          <geometry>
-            <mesh
-              filename="file://$(find my_bot)/description/meshes/base_link.STL" />
-          </geometry>
-          <material
-            name="">
-            <color
-              rgba="0.25098 0.25098 0.25098 1" />
-          </material>
-    </visual>
-    <collision>
-          <origin
-            xyz="0 0 0"
-            rpy="0 0 0" />
-          <geometry>
-            <mesh
-              filename="file://$(find my_bot)/description/meshes/base_link.STL" />
-          </geometry>
+<!-- BASE LINK -->
+  <robot
+  name="Assem 2, Update front plate">
+    <link
+    name="base_link">
+     <inertial>
+       <origin
+        xyz="0.070133662897501 0.00354955354888109 0.0183200114204214"
+        rpy="0 0 0" />
+      <mass
+        value="0.556112519731525" />
+      <inertia
+        ixx="0.00154815109045063"
+        ixy="0.00010780862380031"
+        ixz="0.000221604200759326"
+        iyy="0.0027617246804416"
+        iyz="1.83612061370921E-05"
+        izz="0.00395406219863791" />
+    </inertial>
+    <visual>
+      <origin
+        xyz="0 0 0"
+        rpy="0 0 0" />
+      <geometry>
+        <mesh
+          filename="file://$(find my_bot)/description/meshes/base_link.STL" />
+      </geometry>
+      <material
+        name="">
+        <color
+          rgba="0.250980392156863 0.250980392156863 0.250980392156863 1" />
+      </material>
+    </visual>
+    <collision>
+      <origin
+        xyz="0 0 0"
+        rpy="0 0 0" />
+      <geometry>
+        <mesh
+          filename="file://$(find my_bot)/description/meshes/base_link.STL" />
+      </geometry>
     </collision>
   </link>
@@ -48,41 +51,42 @@
   </gazebo>
  <!-- LEFT WHEEL LINK -->
-  <link name="left_wheel">
-    <inertial>
-          <origin
-            xyz="0 0 -1.3878E-17"
-            rpy="0 0 0" />
-          <mass
-            value="0.10164" />
-          <inertia
-            ixx="3.2133E-05"
-            ixy="3.0279E-19"
-            ixz="3.0269E-21"
-            iyy="5.3678E-05"
-            iyz="-4.2598E-21"
-            izz="3.2133E-05" />
-    </inertial>
-    <visual>
-          <origin
-            xyz="0 0 0"
-            rpy="0 0 0" />
-          <geometry>
-            <mesh
-              filename="file://$(find my_bot)/description/meshes/left_wheel.STL" />
-          </geometry>
-          <material
-            name="">
-            <color
-              rgba="0 0 0.50196 1" />
-          </material>
-    </visual>
-    <collision>
-          <origin
-            xyz="0 0 0"
-            rpy="0 0 0" />
-          <geometry>
-            <mesh
-              filename="file://$(find my_bot)/description/meshes/left_wheel.STL" />
-          </geometry>
+   <link
+    name="left_wheel">
+    <inertial>
+      <origin
+        xyz="6.93889390390723E-18 0 0"
+        rpy="0 0 0" />
+      <mass
+        value="0.10163975077205" />
+      <inertia
+        ixx="3.2132983707622E-05"
+        ixy="3.03239240453886E-19"
+        ixz="-1.94584643807998E-21"
+        iyy="5.36784933764888E-05"
+        iyz="-3.01898169232286E-21"
+        izz="3.2132983707622E-05" />
+    </inertial>
+    <visual>
+      <origin
+        xyz="0 0 0"
+        rpy="0 0 0" />
+      <geometry>
+        <mesh
+          filename="file://$(find my_bot)/description/meshes/left_wheel.STL" />
+      </geometry>
+      <material
+        name="">
+        <color
+          rgba="0 0 0.501960784313725 1" />
+      </material>
+    </visual>
+    <collision>
+      <origin
+        xyz="0 0 0"
+        rpy="0 0 0" />
+      <geometry>
+        <mesh
+          filename="file://$(find my_bot)/description/meshes/left_wheel.STL" />
+      </geometry>
     </collision>
   </link>
@@ -90,7 +94,9 @@
     <material>Gazebo/Blue</material>
   </gazebo>
-  <joint name="left_wheel_joint" type="continuous">
-    <origin
-      xyz="0.001 0.13017 0.0235"
+  <joint
+    name="left_wheel_joint"
+    type="continuous">
+    <origin
+      xyz="0.001 0.12868 0.0235"
       rpy="0 0 0" />
     <parent
@@ -102,19 +108,19 @@
   </joint>
 <!-- RIGHT WHEEL LINK -->
-  <link
+   <link
     name="right_wheel">
     <inertial>
       <origin
-        xyz="6.9389E-18 0 0"
-        rpy="0 0 0" />
-      <mass
-        value="0.10164" />
-      <inertia
-        ixx="3.2133E-05"
-        ixy="-8.6646E-22"
-        ixz="2.1621E-21"
-        iyy="5.3678E-05"
-        iyz="4.6922E-21"
-        izz="3.2133E-05" />
+        xyz="-1.38777878078145E-17 -2.77555756156289E-17 -1.38777878078145E-17"
+        rpy="0 0 0" />
+      <mass
+        value="0.10163975077205" />
+      <inertia
+        ixx="3.2132983707622E-05"
+        ixy="3.0244660672499E-19"
+        ixz="-1.94584643807989E-21"
+        iyy="5.36784933764888E-05"
+        iyz="3.88380233146956E-21"
+        izz="3.2132983707622E-05" />
     </inertial>
     <visual>
@@ -129,5 +135,5 @@
         name="">
         <color
-          rgba="0 0 0.50196 1" />
+          rgba="0 0 0.501960784313725 1" />
       </material>
     </visual>
@@ -149,10 +155,12 @@
     type="continuous">
     <origin
-      xyz="0.001 -0.13017 0.0235"
+      xyz="0.001 -0.12868 0.0235"
       rpy="0 0 0" />
-    <parent link="base_link" />
-    <child link="right_wheel" />
-    <axis
-      xyz="0 1 0" />
+    <parent
+      link="base_link" />
+    <child
+      link="right_wheel" />
+    <axis
+      xyz="0 -1 0" />
   </joint>
 <!-- LIDAR LINK-->
@@ -161,15 +169,15 @@
     <inertial>
       <origin
-        xyz="-0.0067665 9.1926E-05 -0.0083819"
-        rpy="0 0 0" />
-      <mass
-        value="0.17402" />
-      <inertia
-        ixx="8.0412E-05"
-        ixy="-1.0487E-07"
-        ixz="-2.0693E-05"
-        iyy="0.00012563"
-        iyz="4.0429E-07"
-        izz="0.0001436" />
+        xyz="-0.0067665301166636 9.19261110876313E-05 -0.00838187226715975"
+        rpy="0 0 0" />
+      <mass
+        value="0.174023656294632" />
+      <inertia
+        ixx="8.0412346059381E-05"
+        ixy="-1.04874872480737E-07"
+        ixz="-2.06933187729991E-05"
+        iyy="0.000125629651580714"
+        iyz="4.04290059384042E-07"
+        izz="0.000143604492343178" />
     </inertial>
     <visual>
@@ -193,5 +201,5 @@
       <geometry>
         <mesh
-          filename="file://$(find my_bot)/description/meshes/laser_frame.STL" />
+          filename="file://$(find my_bot)/description/meshes/Lidar collision.STL.STL" />
       </geometry>
     </collision>
@@ -204,5 +212,5 @@
     type="fixed">
     <origin
-      xyz="0.1048 0 0.091825"
+      xyz="0.104800054804252 0 0.0820000000000001"
       rpy="0 0 0" />
     <parent
@@ -214,19 +222,19 @@
   </joint>
 <!-- CAMERA LINK-->
-  <link
+    <link
     name="camera_link">
     <inertial>
       <origin
-        xyz="-0.010597 -1.8404E-05 0.0029121"
-        rpy="0 0 0" />
-      <mass
-        value="0.0057972" />
-      <inertia
-        ixx="6.4641E-07"
-        ixy="3.883E-13"
-        ixz="-1.0375E-09"
-        iyy="2.7217E-07"
-        iyz="2.3413E-10"
-        izz="3.8601E-07" />
+        xyz="-0.0103584698596122 -2.01596126545994E-05 0.00163484283690582"
+        rpy="0 0 0" />
+      <mass
+        value="0.00529235477598514" />
+      <inertia
+        ixx="5.17063055319424E-07"
+        ixy="3.88296936830359E-13"
+        ixz="-1.96692485943055E-09"
+        iyy="1.9007613450553E-07"
+        iyz="2.34133392020719E-10"
+        izz="3.37850233450208E-07" />
     </inertial>
     <visual>
@@ -241,14 +249,14 @@
         name="">
         <color
-          rgba="0.25098 0.25098 0.25098 1" />
-      </material>
-    </visual>
-    <collision>
-      <origin
-        xyz="0 0 0"
-        rpy="0 0 0" />
-      <geometry>
-        <mesh
-          filename="file://$(find my_bot)/description/meshes/camera_link.STL" />
+          rgba="0.250980392156863 0.250980392156863 0.250980392156863 1" />
+      </material>
+    </visual>
+    <collision>
+      <origin
+        xyz="0 0 0"
+        rpy="0 0 0" />
+      <geometry>
+        <mesh
+          filename="file://$(find my_bot)/description/meshes/camera collision.STL" />
       </geometry>
     </collision>
@@ -257,9 +265,9 @@
     <material>Gazebo/Orange</material>
   </gazebo>
-  <joint
+   <joint
     name="camera_joint"
     type="fixed">
     <origin
-      xyz="0.16129 0 0.029575"
+      xyz="0.16129 0 0.05345"
       rpy="0 0 0" />
     <parent
@@ -275,15 +283,15 @@
     <inertial>
       <origin
-        xyz="0 1.3878E-17 1.3878E-17"
-        rpy="0 0 0" />
-      <mass
-        value="0.0083657" />
-      <inertia
-        ixx="1.3493E-07"
-        ixy="-4.097E-24"
+        xyz="2.77555756156289E-17 0 1.38777878078145E-17"
+        rpy="0 0 0" />
+      <mass
+        value="0.00836574047989968" />
+      <inertia
+        ixx="1.34931028200302E-07"
+        ixy="-4.09702557397515E-24"
         ixz="0"
-        iyy="1.3493E-07"
-        iyz="5.9132E-39"
-        izz="1.3493E-07" />
+        iyy="1.34931028200302E-07"
+        iyz="5.91319576211689E-39"
+        izz="1.34931028200302E-07" />
     </inertial>
     <visual>
@@ -298,5 +306,5 @@
         name="">
         <color
-          rgba="0.52941 0.54902 0.54902 1" />
+          rgba="0.529411764705882 0.549019607843137 0.549019607843137 1" />
       </material>
     </visual>

Commit message: Fixed error in URDF FILE, added gazebo laser_scan and added RP LIDAR launch file

File: description/robot_core.xacro (robot description, xacro)
@@ -5,6 +5,4 @@
 <robot xmlns:xacro="http://www.ros.org/wiki/xacro">
 <!-- BASE LINK -->
-  <robot
-  name="Assem 2, Update front plate">
     <link
     name="base_link">
@@ -165,6 +163,5 @@
   </joint>
 <!-- LIDAR LINK-->
-  <link
-    name="laser_frame">
+  <link name="laser_frame">
     <inertial>
       <origin
@@ -201,5 +198,5 @@
       <geometry>
         <mesh
-          filename="file://$(find my_bot)/description/meshes/Lidar collision.STL.STL" />
+          filename="file://$(find my_bot)/description/meshes/Lidar collision.STL" />
       </geometry>
     </collision>
@@ -207,4 +204,29 @@
   <gazebo reference="laser_frame">
     <material>Gazebo/Orange</material>
+            <sensor name="laser" type="ray">
+            <pose> 0 0 0 0 0 0 </pose>
+            <visualize>true</visualize>
+            <update_rate>10</update_rate>
+            <ray>
+                <scan>
+                    <horizontal>
+                        <samples>360</samples>
+                        <min_angle>-3.14</min_angle>
+                        <max_angle>3.14</max_angle>
+                    </horizontal>
+                </scan>
+                <range>
+                    <min>0.3</min>
+                    <max>12</max>
+                </range>
+            </ray>
+            <plugin name="laser_controller" filename="libgazebo_ros_ray_sensor.so">
+                <ros>
+                    <argument>~/out:=scan</argument>
+                </ros>
+                <output_type>sensor_msgs/LaserScan</output_type>
+                <frame_name>laser_frame</frame_name>
+            </plugin>
+        </sensor>
   </gazebo>
   <joint
